File: Neopixel_Music_Visualizer.sch (KiCad schematic (older format))
At the start: 15 parts

Commit message: Rail splitter and mono downmixer
Parts:
- C?: value C -> 1uF
- R? (x2): value R -> 1k 1%
- R?: value R -> 200k
- R? (x2): value 1M -> 100k
Connections:
- net +5V: now also U?.8 (V+)
- net GND: now also U?.4 (V-)
- net VGND: now also R?.1
- net INPUT_L: now reaches R?.2
- net INPUT_R: now reaches R?.2
- net at C?.1: now also R?.2, U?.5 (+)
- net MONO_BIASED: now reaches U?.6 (-)
- net MONO_BIASED: now also U?.7
Other:
- note added: "10 frequency bands\n2 opamps per band (non-inverting amp after filter stage, buffer after enveloping stage)\n\n1 opamp at the input for downmixing stereo to mono\n1 opamp as rail splitter"
- note added: "Downmix to mono and add a DC bias"
- note added: "RC high pass filter --> bias to VGND"
- note added: "Rail splitter (virtual ground)"
- note removed: "10 frequency bands\n2 opamps per band (non-inverting amp after filter stage, buffer after enveloping stage)\n1 opamp at the input for downmixing stereo to mono"
- moved on the sheet: C?, R?, U?, U?A, U?B
